File: eagle-schematics/amiga_external_floppy_adapter_rev2_1.sch (EAGLE design)
At the start: 13 parts, among them IC1 74LS00N, IC2 74LS74N, J1 Computer, J2 Floppy, J3 PINHD-1X4, J4 Passthrough

Commit message: Files for rev2.1 are updated/added, readme file modified slightly
Parts:
- added J5: (no value), pinhead:PINHD-1X3
- added J6: (no value), jumper:JP1E
- C1, C2: device rcl:C-EU025-025X050 -> rcl:C-EUC1206
- IC1: value 74LS00N -> 74LS00D; device 74xx-eu:74LS00N -> 74xx-eu:74LS00D
- IC2: value 74LS74N -> 74LS74D; device 74xx-eu:74LS74N -> 74xx-eu:74LS74D
- J3: value PINHD-1X4 -> Power
- R1, R2, R3, R4, R5: device rcl:R-EU_0207/10 -> rcl:R-EU_R1206
Connections:
- new net !SEL: IC1A.I0, IC1A.I1, J2.!SEL0, J5.2, R1.1
- net !MTR: now also J6.1
- net !MTRX: now also J6.2
- net !SEL1: now also J5.3; no longer IC1A.I0, IC1A.I1, J2.!SEL0, R1.1
- net !SEL2: now also J5.1
- net +5V: now also IC1D.I0, IC1D.I1, IC2B.CLK, IC2B.CLR, IC2B.D, IC2B.PRE
- net GND: now also IC1C.I0, IC1C.I1
Other:
- note added: "2.1"
- note added: "Amiga external floppy adapter mod by Sanyi"
- note added: "Nov 15, 2020"
- note removed: "1"
- note removed: "June 29, 2020"
